Commit message: gym ok

File: resources/go2/a1/urdf/a1.urdf (robot description, URDF)
Before this commit: robot a1_description, 23 links, 22 joints
Links:
- link FL_foot: mass 1.5 -> 0.04; geometry collision sphere radius=0.02; visual sphere radius=0.01
- link FR_foot: mass 1.5 -> 0.04; geometry collision sphere radius=0.02; visual sphere radius=0.01
- link RL_foot: mass 1.5 -> 0.04; geometry collision sphere radius=0.02; visual sphere radius=0.01
- link RR_foot: mass 1.5 -> 0.04; geometry visual sphere radius=0.01
Joints:
- removed joint FL_foot_joint
- removed joint FR_foot_joint
- removed joint RL_foot_joint
- removed joint RR_foot_joint
- added joint FL_foot_fixed: type fixed, parent FL_calf, child FL_foot, origin xyz=0 0 -0.2 rpy=0 0 0
- added joint FR_foot_fixed: type fixed, parent FR_calf, child FR_foot, origin xyz=0 0 -0.2 rpy=0 0 0
- added joint RL_foot_fixed: type fixed, parent RL_calf, child RL_foot, origin xyz=0 0 -0.2 rpy=0 0 0
- added joint RR_foot_fixed: type fixed, parent RR_calf, child RR_foot, origin xyz=0 0 -0.2 rpy=0 0 0
- joint RR_hip_joint: origin xyz=-0.26519 -0.0895 -0.0002 rpy=0 0 0 -> xyz=-0.26519 -0.0895 -0.0 rpy=0 0 0

File: resources/titati_urdf/urdf/titatit_robot_2.urdf (robot description, URDF)
Before this commit: robot titatit_robot_2, 21 links, 20 joints
Links:
- link FL_battery: mass 0.86022 -> 1.0E-09
- link FL_thigh: mass 2.06397198838348 -> 3.08318468505764
- link FR_battery: mass 0.86022 -> 1.0E-09
- link RL_battery: mass 0.86022 -> 1.0E-09
- link RR_battery: mass 0.86022 -> 1.0E-09
